File: elec/layout/default/veramonitor.kicad_pcb (KiCad board)
At the start: 2 copper layers, 107.7 x 61.6 mm, 48 parts, among them J1 ?, U1 ?, U10 ?, U11 ?, U12 ?, U13 ?, U14 ?, U15 ?, U16 ?, U17 ?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

Commit message: fixing
Parts:
- removed C1: 50V 10nF X7R ±10% 0402 Multilayer Ceramic Capacitors MLCC -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, lib:C0402
- C10, C11, C12, C13, C14, C4, C8, C9: value 16V 100nF X7R ±10% 0402 Multilayer Ceramic Capacitors MLCC - SMD/SMT ROHS -> 100nF ±10% 16V X7R; footprint lib:C0402 -> atopile:C0402-b3ef17
- C2, C3, C5, C6: value 25V 10uF X5R ±10% 0805 Multilayer Ceramic Capacitors MLCC - SMD/SMT ROHS -> 10µF ±10% 25V X5R; footprint lib:C0805 -> atopile:C0805-3b2e55
- C7: value 6.3V 10uF X5R ±20% 0402 Multilayer Ceramic Capacitors MLCC - SMD/SMT ROHS -> 10µF ±20% 10V X5R; footprint lib:C0402 -> atopile:C0402-b3ef17
- J1, U1, U10, U11, U12, U13, U14, U15, U16, U17, U18, U19, U2, U20, U21, U22, U3, U4, U5, U6, U7, U8, U9: value ? -> (none)
- R1, R2: value 62.5mW Thick Film Resistors 50V ±100ppm/℃ ±1% 4.7kΩ 0402 Chip Resistor - Surface Mount ROHS -> 4.7kΩ ±1% 62.5mW; footprint lib:R0402 -> atopile:R0402-56259e
- R10, R11, R3, R4, R5, R6, R7, R8, R9: value 62.5mW Thick Film Resistors 50V ±100ppm/℃ ±1% 10kΩ 0402 Chip Resistor - Surface Mount ROHS -> 10kΩ ±1% 62.5mW; footprint lib:R0402 -> atopile:R0402-56259e
Connections:
- net backlighten renamed BL
- net bclk renamed BCLK
- net cc1 renamed CC1
- net cc2 renamed B5
- net din renamed DIN
- net dummy renamed DUMMY
- net en renamed in
- net gain_slot renamed GAIN_SLOT
- net io14 renamed KEY-1
- net io16 renamed DIN-1
- net io21 renamed KEY-2
- net io35 renamed KEY
- net io45 renamed KEY-4
- net io47 renamed KEY-5
- net io48 renamed KEY-3
- net jtag_connector-reset renamed reset
- net lrclk renamed LRCLK
- net micro.ic-reset renamed RST
- net micro.ic-vcc renamed in-1
- net n_period_c_period renamed N_period_C_period
- net outn renamed OUTN
- net outp renamed OUTP
- net rxd0 renamed rx
- net sd_mode_hash renamed SD_MODE_hash
- net sub1 renamed SUB1
- net sub2 renamed B8
- net sw1-dout renamed io
- net sw3-dout renamed io-1
- net sw4-dout renamed io-2
- net sw6-dout renamed DOUT
- net txd0 renamed tx
- C10 pad 1: vcc-1 -> hv
- C11 pad 1: vcc-1 -> hv
- C12 pad 1: vcc-1 -> hv
- C13 pad 1: vcc-1 -> hv
- C14 pad 1: vcc-1 -> hv
- C2 pad 1: vcc -> hv-1
- C3 pad 1: vcc-1 -> hv
- C4 pad 1: vcc-1 -> hv
- C5 pad 1: vcc-1 -> hv
- C6 pad 1: vcc-1 -> hv
- C7 pad 1: vcc-1 -> hv
- C8 pad 1: vcc-1 -> hv
- C9 pad 1: vcc-1 -> hv
- J1 pad 2: vcc-1 -> hv
- R10 pad 1: vcc-1 -> hv
- R11 pad 1: vcc-1 -> hv
- R3 pad 1: vcc-1 -> hv
- R4 pad 1: vcc-1 -> hv
- R5 pad 1: vcc-1 -> hv
- R6 pad 1: vcc-1 -> hv
- R7 pad 1: vcc-1 -> hv
- R8 pad 1: vcc-1 -> hv
- R9 pad 1: vcc-1 -> hv
- U1 pad 1: vcc -> hv-1
- U11 pad 1: vcc-1 -> hv
- U11 pad 2: sw2-dout -> vcc
- U13 pad 1: vcc-1 -> hv
- U13 pad 4: sw2-dout -> vcc
- U15 pad 1: vcc-1 -> hv
- U17 pad 1: vcc-1 -> hv
- U17 pad 2: sw5-dout -> vcc-1
- U19 pad 1: vcc-1 -> hv
- U19 pad 4: sw5-dout -> vcc-1
- U2 pad A4: vcc -> hv-1
- U2 pad A9: vcc -> hv-1
- U2 pad B4: vcc -> hv-1
- U2 pad B9: vcc -> hv-1
- U3 pad 5: vcc-1 -> hv
- U4 pad 2: vcc-1 -> hv
- U4 pad 3: vcc -> hv-1
- U4 pad 4: vcc-1 -> hv
- U5 pad 18: dc -> cs
- U5 pad 19: cs -> mosi
- U5 pad 2: vcc-1 -> hv
- U5 pad 21: mosi -> miso
- U7 pad 1: vcc -> hv-1
- U7 pad 3: mosi -> miso
- U7 pad 5: cs -> mosi
- U7 pad 6: dc -> cs
- U8 pad 7: vcc-1 -> hv
- U8 pad 8: vcc-1 -> hv
- U9 pad 1: vcc-1 -> hv
Routing:
- net hv: track 0.00 -> 373.9 mm, vias 0 -> 13
- net vcc-1: track 373.9 -> 25.0 mm, vias 13 -> 2
- net hv-1: track 0.00 -> 104.3 mm, vias 0 -> 4
- net vcc: track 104.3 -> 17.8 mm, vias 4 -> 2
- net sw5-dout: track 25.0 -> 0.00 mm, vias 2 -> 0
- net sw2-dout: track 17.8 -> 0.00 mm, vias 2 -> 0
- net dc: track 7.97 -> 0.00 mm
- net miso: track 0.00 -> 6.71 mm
- net mosi: track 6.71 -> 7.64 mm
Other:
- board outline removed
- board text removed: "izzymonitor :3"
