File: elec/layout/kailh-sw/kailh-sw.kicad_pcb (KiCad board)
At the start: 2 copper layers, 40 x 40 mm, 4 parts, among them U1 100nF ±10% 16V X7R, U3 10kΩ ±1% 62.5mW

Commit message: fixing
Parts:
- moved U4 40.3 mm to (0.00, 0.00)
- moved U1 20.6 mm to (10.0, 0.00)
- moved U3 20.6 mm to (0.00, -10.0)
- moved U2 5.00 mm to (10.0, -10.0)
Other:
- board outline removed
- board text removed: "{{GITHASH}}"
